File: PowerSupply/PowerSupply.kicad_pcb (KiCad board)
At the start: 2 copper layers, 100 x 100 mm, 64 parts, among them J1 Conn_01x01, J2 Conn_01x01, J3 Conn_01x01, J4 Conn_01x05, J5 Conn_01x04, J6 Conn_01x04, J7 Conn_01x16, J8 Conn_01x01, J9 Conn_01x01, U1 LM358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

Commit message: aaa
Parts:
- moved C14 27.2 mm to (60.9, 82.3)
- moved J8 27.2 mm to (53.4, 64.0)
- moved J9 27.2 mm to (53.4, 57.0)
- moved C1 27.2 mm to (55.2, 70.0)
- moved C10 27.2 mm to (65.6, 79.6)
- moved C12 27.2 mm to (68.7, 82.8)
- moved C13 27.2 mm to (77.4, 61.5)
- moved C15 27.2 mm to (71.8, 79.7)
- moved C16 27.2 mm to (79.9, 97.2)
- moved C17 27.2 mm to (79.9, 93.1)
- moved C18 27.2 mm to (74.3, 95.5)
- moved C19 27.2 mm to (74.3, 91.5)
- moved C2 27.2 mm to (64.9, 69.9)
- moved C20 27.2 mm to (83.3, 97.2)
- moved C21 27.2 mm to (83.3, 93.1)
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Routing:
- net +5V: track 93.5 -> 86.9 mm, vias 2 -> 3
- net GND: vias 12 -> 13
Other:
- board size 100 x 100 mm -> 43 x 60 mm

Commit message: update
Parts:
- added C24: CP, Capacitor_THT:CP_Radial_D6.3mm_P2.50mm, F.Cu at (92.9, 72.9)
- C13: value 10u -> 1u
- moved C10 28.7 mm to (91.0, 93.0)
- moved C11 28.7 mm to (80.0, 95.7)
- moved C13 28.7 mm to (102.8, 74.9)
- moved C18 28.7 mm to (99.7, 108.9)
- moved C19 28.7 mm to (99.7, 104.9)
- moved C21 28.7 mm to (108.7, 106.5)
- moved C22 28.7 mm to (78.7, 101.5)
- moved C23 28.7 mm to (91.7, 109.5)
- moved C29 28.7 mm to (107.7, 101.2)
- moved C4 28.7 mm to (105.9, 85.2)
- moved C7 28.7 mm to (100.4, 78.5)
- moved C9 28.7 mm to (95.4, 81.4)
- moved D1 28.7 mm to (98.2, 72.0)
- moved J2 28.7 mm to (115.4, 70.4)
- moved J3 28.7 mm to (115.4, 77.4)
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Routing:
- net +24V: track 43.8 -> 53.6 mm
- net GPIO_PB1: track 22.1 -> 24.2 mm
- net Iout: track 44.0 -> 45.6 mm
- net GND: track 18.8 -> 20.4 mm, vias 13 -> 35
- net TIM3_CH1: track 26.1 -> 27.2 mm
- net +3V3: track 86.0 -> 86.8 mm
- net (no net): vias 0 -> 4
Other:
- board size 43 x 60 mm -> 56 x 61 mm
- net class Default: clearance 0.254 -> 0.2032
- rule trace_clearance: 0.254 -> 0.2032
- board text added: "+"
- board text added: "+ OUT"
- board text added: "-"
- board text added: "- OUT"
- board text added: "Daniel Hert 2019"
- board text added: "Supply V4"
- board text added: "V_Sense"
