File: PowerSupply/PowerSupply.sch (KiCad schematic (older format))
At the start: 26 parts

Commit message: updat
Parts:
- added C?: 100n, symbol Device:C
- added C? (x3): 1u, symbol Device:C
- added U?: TPS60403, Package_TO_SOT_SMD:SOT-23-5, symbol PowerSupply:TPS60403
Connections:
- net +5V is gone; now on net +24V: U?.8 (V+)
- net +24V: now also C?.1
- net +3.3VA: now also C?.2, U?.2 (IN)
- net GND: now also U?.1 (REF), U?.2 (GND), C?.1, C?.1, C?.2, U?.4 (GND); no longer U?.4 (V-)
- net at D?.1, R?.2, U?.7: now also C?.1
- new net: C?.1, U?.3 (C_FLY-)
- new net: C?.2, U?.5 (C_FLY+)
- new net -3V3: C?.2, U?.1 (OUT), U?.4 (V-)
Changed lines of the file:
@@
 EESchema Schematic File Version 4
 LIBS:PowerSupply-cache
-EELAYER 30 0
+EELAYER 29 0
 EELAYER END
 $Descr A4 11693 8268
@@
 Wire Wire Line
 	4750 2250 4750 1950
-$Comp
-L power:+5V #PWR?
-U 1 1 5D722B01
-P 3600 2050
-F 0 "#PWR?" H 3600 1900 50  0001 C CNN
-F 1 "+5V" H 3615 2223 50  0000 C CNN
-F 2 "" H 3600 2050 50  0001 C CNN
-F 3 "" H 3600 2050 50  0001 C CNN
-	1    3600 2050
-	1    0    0    -1
-$EndComp
-Wire Wire Line
-	3600 2050 3600 2150
 Wire Wire Line
 	5150 2450 5050 2450
@@
 	-1   0    0    1
 $EndComp
-Wire Wire Line
-	2700 3000 2700 2950
-Connection ~ 2700 3000
-Wire Wire Line
-	3000 3000 3000 2950
-Wire Wire Line
-	2700 3000 3000 3000
-Wire Wire Line
-	2700 3050 2700 3000
 $Comp
 L power:GND #PWR?
@@
 $EndComp
 Wire Wire Line
-	3000 2550 2700 2550
-Connection ~ 3000 2550
-Wire Wire Line
-	3000 2650 3000 2550
-Wire Wire Line
 	2700 2550 2600 2550
 Connection ~ 2700 2550
 Wire Wire Line
 	2700 2650 2700 2550
-$Comp
-L Device:C C?
-U 1 1 5D71E052
-P 3000 2800
-F 0 "C?" H 3115 2846 50  0000 L CNN
-F 1 "1n" H 3115 2755 50  0000 L CNN
-F 2 "" H 3038 2650 50  0001 C CNN
-F 3 "~" H 3000 2800 50  0001 C CNN
-	1    3000 2800
-	1    0    0    -1
-$EndComp
 $Comp
 L Device:R R?
@@
 $Comp
 L Amplifier_Operational:LM358 U?
-U 3 1 5D7083D0
-P 3700 2450
-F 0 "U?" H 3658 2496 50  0000 L CNN
-F 1 "LM358" H 3658 2405 50  0000 L CNN
-F 2 "" H 3700 2450 50  0001 C CNN
-F 3 "http://www.ti.com/lit/ds/symlink/lm2904-n.pdf" H 3700 2450 50  0001 C CNN
-	3    3700 2450
-	1    0    0    -1
-$EndComp
-$Comp
-L Amplifier_Operational:LM358 U?
 U 2 1 5D70610A
 P 4050 3750
@@
 F 3 "http://www.ti.com/lit/ds/symlink/lm2904-n.pdf" H 4050 3750 50  0001 C CNN
 	2    4050 3750
-	1    0    0    -1
-$EndComp
-$Comp
-L Amplifier_Operational:LM358 U?
-U 1 1 5D704E8C
-P 3700 2450
-F 0 "U?" H 3800 2750 50  0000 C CNN
-F 1 "LM358" H 3800 2650 50  0000 C CNN
-F 2 "" H 3700 2450 50  0001 C CNN
-F 3 "http://www.ti.com/lit/ds/symlink/lm2904-n.pdf" H 3700 2450 50  0001 C CNN
-	1    3700 2450
 	1    0    0    -1
 $EndComp
@@
 $Comp
 L Device:C C?
-U 1 1 5D7218D0
-P 3900 3000
-F 0 "C?" H 4015 3046 50  0000 L CNN
-F 1 "1n" H 4015 2955 50  0000 L CNN
-F 2 "" H 3938 2850 50  0001 C CNN
-F 3 "~" H 3900 3000 50  0001 C CNN
-	1    3900 3000
-	0    1    1    0
-$EndComp
-Wire Wire Line
-	4050 3000 4150 3000
-Wire Wire Line
-	4150 3000 4150 2450
-Wire Wire Line
-	4000 2450 4150 2450
-Wire Wire Line
-	4150 2450 4450 2450
-Connection ~ 4150 2450
-$Comp
-L Device:C C?
 U 1 1 5D7322D1
 P 2450 2150
@@
 Wire Wire Line
 	2200 2550 2300 2550
-Wire Wire Line
-	3000 2550 3300 2550
-Wire Wire Line
-	3300 2550 3300 3000
-Connection ~ 3300 2550
-Wire Wire Line
-	3300 2550 3400 2550
-Wire Wire Line
-	3300 3000 3750 3000
-$Comp
-L power:GND #PWR?
-U 1 1 5D74C0FE
-P 3600 2750
-F 0 "#PWR?" H 3600 2500 50  0001 C CNN
-F 1 "GND" H 3605 2577 50  0000 C CNN
-F 2 "" H 3600 2750 50  0001 C CNN
-F 3 "" H 3600 2750 50  0001 C CNN
-	1    3600 2750
-	1    0    0    -1
-$EndComp
 $Comp
 L Device:C C?
@@
 	3550 4150 3850 4150
 Wire Wire Line
-	4200 4150 4450 4150
-Wire Wire Line
 	4450 4150 4450 3750
 Connection ~ 4450 3750
@@
 	3750 3850 3550 3850
 Connection ~ 3550 3850
-Text GLabel 3250 2350 0    50   Input ~ 0
-V_SET
-Wire Wire Line
-	3250 2350 3400 2350
 Text GLabel 3550 3650 0    50   Input ~ 0
 I_SET
@@
 Wire Wire Line
 	9600 1750 9600 1650
+Connection ~ 2700 3000
+Wire Wire Line
+	2700 3050 2700 3000
+Wire Wire Line
+	2700 3000 2700 2950
+Wire Wire Line
+	3250 2350 3400 2350
+Text GLabel 3250 2350 0    50   Input ~ 0
+V_SET
+Wire Wire Line
+	3300 3000 3750 3000
+Wire Wire Line
+	3300 2550 3400 2550
+Connection ~ 3300 2550
+Wire Wire Line
+	3300 2550 3300 3000
+Wire Wire Line
+	3000 2550 3300 2550
+Wire Wire Line
+	4000 2450 4150 2450
+Wire Wire Line
+	4150 3000 4150 2450
+Wire Wire Line
+	4050 3000 4150 3000
+$Comp
+L Device:C C?
+U 1 1 5D7218D0
+P 3900 3000
+F 0 "C?" H 4015 3046 50  0000 L CNN
+F 1 "1n" H 4015 2955 50  0000 L CNN
+F 2 "" H 3938 2850 50  0001 C CNN
+F 3 "~" H 3900 3000 50  0001 C CNN
+	1    3900 3000
+	0    1    1    0
+$EndComp
+$Comp
+L Amplifier_Operational:LM358 U?
+U 1 1 5D704E8C
+P 3700 2450
+F 0 "U?" H 3800 2750 50  0000 C CNN
+F 1 "LM358" H 3800 2650 50  0000 C CNN
+F 2 "" H 3700 2450 50  0001 C CNN
+F 3 "http://www.ti.com/lit/ds/symlink/lm2904-n.pdf" H 3700 2450 50  0001 C CNN
+	1    3700 2450
+	1    0    0    -1
+$EndComp
+$Comp
+L Amplifier_Operational:LM358 U?
+U 3 1 5D7083D0
+P 3700 2450
+F 0 "U?" H 3658 2496 50  0000 L CNN
+F 1 "LM358" H 3658 2405 50  0000 L CNN
+F 2 "" H 3700 2450 50  0001 C CNN
+F 3 "http://www.ti.com/lit/ds/symlink/lm2904-n.pdf" H 3700 2450 50  0001 C CNN
+	3    3700 2450
+	1    0    0    -1
+$EndComp
+$Comp
+L Device:C C?
+U 1 1 5D71E052
+P 3000 2800
+F 0 "C?" H 3115 2846 50  0000 L CNN
+F 1 "1n" H 3115 2755 50  0000 L CNN
+F 2 "" H 3038 2650 50  0001 C CNN
+F 3 "~" H 3000 2800 50  0001 C CNN
+	1    3000 2800
+	1    0    0    -1
+$EndComp
+Wire Wire Line
+	3000 2650 3000 2550
+Connection ~ 3000 2550
+Wire Wire Line
+	3000 2550 2700 2550
+Wire Wire Line
+	2700 3000 3000 3000
+Wire Wire Line
+	3000 3000 3000 2950
+Wire Wire Line
+	4150 2450 4450 2450
+Connection ~ 4150 2450
+Wire Wire Line
+	4150 4150 4450 4150
+$Comp
+L power:GND #PWR?
+U 1 1 5D72CBEF
+P 8400 2500
+F 0 "#PWR?" H 8400 2250 50  0001 C CNN
+F 1 "GND" H 8405 2327 50  0000 C CNN
+F 2 "" H 8400 2500 50  0001 C CNN
+F 3 "" H 8400 2500 50  0001 C CNN
+	1    8400 2500
+	1    0    0    -1
+$EndComp
+Wire Wire Line
+	7950 2300 8050 2300
+Wire Wire Line
+	8400 2500 8400 2450
+Wire Wire Line
+	8400 2450 7950 2450
+Wire Wire Line
+	7950 2300 7950 2450
+Wire Wire Line
+	8400 2450 8850 2450
+Wire Wire Line
+	8850 2450 8850 2300
+Wire Wire Line
+	8850 2300 8750 2300
+Connection ~ 8400 2450
+$Comp
+L power:+24V #PWR?
+U 1 1 5D7356D4
+P 3600 1900
+F 0 "#PWR?" H 3600 1750 50  0001 C CNN
+F 1 "+24V" H 3615 2073 50  0000 C CNN
+F 2 "" H 3600 1900 50  0001 C CNN
+F 3 "" H 3600 1900 50  0001 C CNN
+	1    3600 1900
+	1    0    0    -1
+$EndComp
+$Comp
+L Device:C C?
+U 1 1 5D735CD6
+P 3850 2000
+F 0 "C?" H 3965 2046 50  0000 L CNN
+F 1 "100n" H 3965 1955 50  0000 L CNN
+F 2 "" H 3888 1850 50  0001 C CNN
+F 3 "~" H 3850 2000 50  0001 C CNN
+	1    3850 2000
+	0    -1   -1   0
+$EndComp
+Wire Wire Line
+	3700 2000 3600 2000
+Wire Wire Line
+	3600 2000 3600 2150
+Wire Wire Line
+	3600 2000 3600 1900
+Connection ~ 3600 2000
+$Comp
+L power:GND #PWR?
+U 1 1 5D73CA0D
+P 4100 2100
+F 0 "#PWR?" H 4100 1850 50  0001 C CNN
+F 1 "GND" H 4105 1927 50  0000 C CNN
+F 2 "" H 4100 2100 50  0001 C CNN
+F 3 "" H 4100 2100 50  0001 C CNN
+	1    4100 2100
+	1    0    0    -1
+$EndComp
+Wire Wire Line
+	4100 2100 4100 2000
+Wire Wire Line
+	4100 2000 4000 2000
+$Comp
+L power:-3V3 #PWR?
+U 1 1 5D740108
+P 3600 2750
+F 0 "#PWR?" H 3600 2850 50  0001 C CNN
+F 1 "-3V3" H 3615 2923 50  0000 C CNN
+F 2 "" H 3600 2750 50  0001 C CNN
+F 3 "" H 3600 2750 50  0001 C CNN
+	1    3600 2750
+	-1   0    0    1
+$EndComp
+$Comp
+L PowerSupply:TPS60403 U?
+U 1 1 5D7415CA
+P 3300 5600
+F 0 "U?" H 3300 5925 50  0000 C CNN
+F 1 "TPS60403" H 3300 5834 50  0000 C CNN
+F 2 "Package_TO_SOT_SMD:SOT-23-5" H 3200 5300 50  0001 C CNN
+F 3 "" H 3300 5150 50  0001 C CNN
+	1    3300 5600
+	1    0    0    -1
+$EndComp
+$Comp
+L power:+3.3VA #PWR?
+U 1 1 5D743004
+P 2200 5400
+F 0 "#PWR?" H 2200 5250 50  0001 C CNN
+F 1 "+3.3VA" H 2215 5573 50  0000 C CNN
+F 2 "" H 2200 5400 50  0001 C CNN
+F 3 "" H 2200 5400 50  0001 C CNN
+	1    2200 5400
+	1    0    0    -1
+$EndComp
+$Comp
+L Device:C C?
+U 1 1 5D7472D7
+P 2700 5800
+F 0 "C?" H 2815 5846 50  0000 L CNN
+F 1 "1u" H 2815 5755 50  0000 L CNN
+F 2 "" H 2738 5650 50  0001 C CNN
+F 3 "~" H 2700 5800 50  0001 C CNN
+	1    2700 5800
+	-1   0    0    1
+$EndComp
+Wire Wire Line
+	2200 5400 2200 5500
+Connection ~ 2200 5500
+$Comp
+L Device:C C?
+U 1 1 5D75220E
+P 4100 5850
+F 0 "C?" H 4215 5896 50  0000 L CNN
+F 1 "1u" H 4215 5805 50  0000 L CNN
+F 2 "" H 4138 5700 50  0001 C CNN
+F 3 "~" H 4100 5850 50  0001 C CNN
+	1    4100 5850
+	-1   0    0    1
+$EndComp
+Wire Wire Line
+	3700 5700 3800 5700
+Wire Wire Line
+	4100 5500 3700 5500
+$Comp
+L power:GND #PWR?
+U 1 1 5D75A118
+P 3800 6150
+F 0 "#PWR?" H 3800 5900 50  0001 C CNN
+F 1 "GND" H 3805 5977 50  0000 C CNN
+F 2 "" H 3800 6150 50  0001 C CNN
+F 3 "" H 3800 6150 50  0001 C CNN
+	1    3800 6150
+	1    0    0    -1
+$EndComp
+$Comp
+L Device:C C?
+U 1 1 5D76C1EF
+P 2200 5800
+F 0 "C?" H 2315 5846 50  0000 L CNN
+F 1 "1u" H 2315 5755 50  0000 L CNN
+F 2 "" H 2238 5650 50  0001 C CNN
+F 3 "~" H 2200 5800 50  0001 C CNN
+	1    2200 5800
+	-1   0    0    1
+$EndComp
+Wire Wire Line
+	2900 5600 2700 5600
+Wire Wire Line
+	2700 5600 2700 5650
+Wire Wire Line
+	2900 5700 2850 5700
+Wire Wire Line
+	2850 5700 2850 6000
+Wire Wire Line
+	2850 6000 2700 6000
+Wire Wire Line
+	2700 6000 2700 5950
+Wire Wire Line
+	2200 5950 2200 6050
+Wire Wire Line
+	2200 6050 3800 6050
+Wire Wire Line
+	4100 6050 4100 6000
+Wire Wire Line
+	3800 6150 3800 6050
+Connection ~ 3800 6050
+Wire Wire Line
+	3800 6050 4100 6050
+Wire Wire Line
+	3800 5700 3800 6050
+Wire Wire Line
+	4100 5500 4100 5700
+Wire Wire Line
+	2200 5500 2900 5500
+Wire Wire Line
+	2200 5500 2200 5650
+$Comp
+L power:-3V3 #PWR?
+U 1 1 5D78E542
+P 4100 5400
+F 0 "#PWR?" H 4100 5500 50  0001 C CNN
+F 1 "-3V3" H 4115 5573 50  0000 C CNN
+F 2 "" H 4100 5400 50  0001 C CNN
+F 3 "" H 4100 5400 50  0001 C CNN
+	1    4100 5400
+	1    0    0    -1
+$EndComp
+Wire Wire Line
+	4100 5400 4100 5500
+Connection ~ 4100 5500
 $EndSCHEMATC

Commit message: updaaaat
Parts:
- removed C?: 1n, symbol Device:C
- removed Q? (x3): Q_NPN_BCE, symbol Device:Q_NPN_BCE
- removed R?: R, symbol Device:R
- removed R?: 68R, symbol Device:R
- removed R?: 13K, symbol Device:R
- removed U?: INA210, symbol PowerSupply:INA210
- removed U?: STM32F042K6Tx, Package_QFP:LQFP-32_7x7mm_P0.8mm, symbol MCU_ST_STM32F0:STM32F042K6Tx
- removed U?: TPS60403, Package_TO_SOT_SMD:SOT-23-5, symbol PowerSupply:TPS60403
- added C1, C2, C22, C23, C25, C26, C27, C28, C29, C5: 100n, Capacitor_SMD:C_0805_2012Metric, symbol Device:C
- added C11, C16, C17, C20, C21: 1u, Capacitor_SMD:C_0805_2012Metric, symbol Device:C
- added C14: 330p, Capacitor_SMD:C_0805_2012Metric, symbol Device:C
- added C18, C19: 20p, Capacitor_SMD:C_0805_2012Metric, symbol Device:C
- added J1: Conn_01x01, Connector_Wire:SolderWirePad_1x01_Drill0.8mm, symbol Connector_Generic:Conn_01x01
- added J4: Conn_01x05, Connector_PinHeader_2.54mm:PinHeader_1x05_P2.54mm_Vertical, symbol Connector_Generic:Conn_01x05
- added J5, J6: Conn_01x04, Connector_PinSocket_2.54mm:PinSocket_1x04_P2.54mm_Vertical, symbol Connector_Generic:Conn_01x04
- added J7: Conn_01x16, Connector_PinSocket_2.54mm:PinSocket_1x16_P2.54mm_Vertical, symbol Connector_Generic:Conn_01x16
- added J8, J9: Conn_01x01, Connector_Wire:SolderWirePad_1x01_Drill2mm, symbol Connector_Generic:Conn_01x01
- added R10, R6, R7, R8, R9: 13K, Resistor_SMD:R_0805_2012Metric, symbol Device:R
- added R11, R14, R15, R16, R17: 0R05, Resistor_SMD:R_1206_3216Metric, symbol Device:R
- added R12, R13: NoPopulate!, Resistor_SMD:R_0805_2012Metric, symbol Device:R
- added U1, U9: LM358, Package_SO:SOIC-8_3.9x4.9mm_P1.27mm, symbol Amplifier_Operational:LM358
- added U2: L7805, Package_TO_SOT_SMD:TO-252-2, symbol Regulator_Linear:L7805
- added U5: MCP1501T-33E_CHY, Package_TO_SOT_SMD:SOT-23-6, symbol PowerSupplyLib:MCP1501T-33E_CHY
- added U6: TPS60403, Package_TO_SOT_SMD:SOT-23-5, symbol PowerSupplyLib:TPS60403
- added U7: INA213, Package_TO_SOT_SMD:SOT-363_SC-70-6_Handsoldering, symbol PowerSupplyLib:INA210
- added U8: STM32F030K6Tx, Package_QFP:LQFP-32_7x7mm_P0.8mm, symbol MCU_ST_STM32F0:STM32F030K6Tx
- added Y1: Crystal32MHz, Crystal:Crystal_HC49-U_Vertical, symbol Device:Crystal
- C10, C12, C13, C15, C3, C4, C6, C7, C8, C9: renamed from C?; footprint (none) -> Capacitor_SMD:C_0805_2012Metric
- J2, J3: renamed from J?; footprint (none) -> Connector_Wire:SolderWirePad_1x01_Drill2mm
- R1, R2, R3: renamed from R?; footprint (none) -> Resistor_SMD:R_0805_2012Metric
- R4: renamed from R?; value 13K -> 250R; footprint (none) -> Resistor_SMD:R_0805_2012Metric
- U3: renamed from U?; footprint (none) -> Package_SO:SOIC-8_3.9x4.9mm_P1.27mm
- U4: renamed from U?; footprint (none) -> Package_TO_SOT_THT:TO-220-3_Vertical
- gave numbers to parts that had none: 1
Connections:
- net +24V: now also C1.1, J9.1 (Pin_1), U2.1 (IN)
- net +3.3VA: now also C14.2, C25.1, C27.1, R12.1, U1.3 (+), U1.5 (+), U5.1 (OUT), U7.3 (V+), U8.5 (VDDA); no longer C10.2
- net -3V3: now also C28.1, C29.1, U6.1 (OUT), U9.4 (V-)
- net GND: now also C1.2, C11.1, C14.1, C16.1, C17.1, C18.1, C19.1, C2.2, C20.1, C21.1, C22.2, C23.2, C25.2, C26.2, C27.2, C28.2, C29.2, C5.2, J4.5 (Pin_5), J6.1 (Pin_1), J6.2 (Pin_2), J6.3 (Pin_3), J6.4 (Pin_4), J8.1 (Pin_1), R8.1, U1.4 (V-), U2.2 (GND), U5.2 (GND), U5.3 (GND), U5.4 (~SHDN), U5.5 (GND), U6.4 (GND), U7.1 (REF), U7.2 (GND), U8.16 (VSS), U8.32 (VSS)
- net I_SET: now also U3.3 (+), C21.2, R10.1; no longer U3.5 (+)
- net Iout: now also U7.6 (OUT), U9.3 (+)
- net V_SET: now also U3.5 (+), C20.2, R9.1; no longer U3.3 (+)
- net Vout: now also J1.1 (Pin_1); no longer J2.1 (Pin_1)
- net at D1.3, U4.1 (ADJ): now also R4.1
- net at C13.1, R4.2, U4.2 (VO): now also R11.2, R14.2, R15.2, R16.2, R17.2, U7.4 (IN+)
- net at C8.1, D1.2: now also U3.7; no longer U3.1
- net Vmes: now reaches C3.1, C4.1, C8.2, R1.1, R2.2
- net Vmes: now also U3.6 (-), U9.5 (+); no longer U3.2 (-)
- net at C6.1, C9.2, R3.1: now also U3.2 (-); no longer U3.6 (-)
- net at C9.1, D1.1: now also U3.1; no longer U3.7
- net at C12.1: now also U6.3 (C_FLY-)
- net at C12.2: now also U6.5 (C_FLY+)
- new net: J2.1 (Pin_1), R11.1, R14.1, R15.1, R16.1, R17.1, U7.5 (IN-)
- new net: U8.6 (PA0), U9.1, U9.2 (-)
- new net: U8.7 (PA1), U9.6 (-), U9.7
- new net: C18.2, U8.2 (PF0), Y1.1
- new net: C19.2, U8.3 (PF1), Y1.2
- new net: R8.2, U8.31 (BOOT0)
- new net: J4.4 (Pin_4), R13.2
- new net: C16.2, R6.1, R9.2
- new net: C17.2, R10.2, R7.1
- new net +3V3: C10.2, C22.1, C23.1, J5.1 (Pin_1), J5.2 (Pin_2), R12.2, R13.1, U1.1, U1.2 (-), U1.6 (-), U1.7, U6.2 (IN), U8.1 (VDD), U8.17 (VDD)
- new net +5V: C11.2, C2.1, C26.1, C5.1, J5.3 (Pin_3), J5.4 (Pin_4), U1.8 (V+), U2.3 (OUT), U5.6 (V_DD), U9.8 (V+)
- new net GPIO_PA11: J7.10 (Pin_10), U8.21 (PA11)
- new net GPIO_PA12: J7.11 (Pin_11), U8.22 (PA12)
- new net GPIO_PA15: J7.12 (Pin_12), U8.25 (PA15)
- new net GPIO_PA4: J7.7 (Pin_7), U8.10 (PA4)
- new net GPIO_PA8: J7.6 (Pin_6), U8.18 (PA8)
- new net GPIO_PB1: J7.16 (Pin_16), U8.15 (PB1)
- new net GPIO_PB3: J7.15 (Pin_15), U8.26 (PB3)
- new net GPIO_PB6: J7.14 (Pin_14), U8.29 (PB6)
- new net GPIO_PB7: J7.13 (Pin_13), U8.30 (PB7)
- new net I2C_SCL: J7.8 (Pin_8), U8.19 (PA9)
- new net I2C_SDA: J7.9 (Pin_9), U8.20 (PA10)
- new net NRST: J4.3 (Pin_3), U8.4 (NRST)
- new net SPI_MISO: J7.4 (Pin_4), U8.12 (PA6)
- new net SPI_MOSI: J7.5 (Pin_5), U8.13 (PA7)
- new net SPI_SCK: J7.3 (Pin_3), U8.11 (PA5)
- new net SWCLK: J4.2 (Pin_2), U8.24 (PA14)
- new net SWDIO: J4.1 (Pin_1), U8.23 (PA13)
- new net TIM3_CH1: R6.2, U8.27 (PB4)
- new net TIM3_CH2: R7.2, U8.28 (PB5)
- new net USART_RX: J7.2 (Pin_2), U8.9 (PA3)
- new net USART_TX: J7.1 (Pin_1), U8.8 (PA2)
Other:
- note added: "Krystal\nhttps://www.tme.eu/cz/details/32.00m-hc49-s/krystalove-rezonatory-tht/yic/\n\nRezistor\nhttps://www.tme.eu/cz/details/oar1r010flf/rezistory-1w/tt-electronics/\n"
- note removed: "STM32G070CBT6"
- moved on the sheet: C10, C12, C13, C15, C8, R4, U3A, U3B

Commit message: update
Parts:
- added C24: CP, Capacitor_THT:CP_Radial_D6.3mm_P2.50mm, symbol Device:CP
- C13: value 10u -> 1u
Connections:
- net +24V: now also C24.1
- net GND: now also C24.2
Changed lines of the file:
@@
 P 6150 1900
 F 0 "C13" H 6265 1946 50  0000 L CNN
-F 1 "10u" H 6265 1855 50  0000 L CNN
+F 1 "1u" H 6265 1855 50  0000 L CNN
 F 2 "Capacitor_SMD:C_0805_2012Metric" H 6188 1750 50  0001 C CNN
 F 3 "~" H 6150 1900 50  0001 C CNN
@@
 $EndComp
 Wire Wire Line
-	4450 1650 3750 1650
+	4450 1650 4250 1650
 Wire Wire Line
 	3750 1650 3750 1550
@@
 Wire Wire Line
 	8600 1650 9750 1650
+$Comp
+L Device:CP C24
+U 1 1 5D890238
+P 4250 1850
+F 0 "C24" H 4368 1896 50  0000 L CNN
+F 1 "CP" H 4368 1805 50  0000 L CNN
+F 2 "Capacitor_THT:CP_Radial_D6.3mm_P2.50mm" H 4288 1700 50  0001 C CNN
+F 3 "~" H 4250 1850 50  0001 C CNN
+	1    4250 1850
+	1    0    0    -1
+$EndComp
+$Comp
+L power:GND #PWR0151
+U 1 1 5D89135D
+P 4250 2000
+F 0 "#PWR0151" H 4250 1750 50  0001 C CNN
+F 1 "GND" H 4255 1827 50  0000 C CNN
+F 2 "" H 4250 2000 50  0001 C CNN
+F 3 "" H 4250 2000 50  0001 C CNN
+	1    4250 2000
+	1    0    0    -1
+$EndComp
+Wire Wire Line
+	4250 1700 4250 1650
+Connection ~ 4250 1650
+Wire Wire Line
+	4250 1650 3750 1650
 $EndSCHEMATC
